File: dreaeduino.kicad_pcb (KiCad board)
At the start: 2 copper layers, 48.3 x 55.9 mm, 22 parts, among them J1 Conn_01x08_Female, J2 Conn_01x08_Female, J3 Conn_01x08_Female, J4 Conn_01x08_Female, J5 USB_B_Micro, J6 Conn_02x03_Odd_Even, J7 Conn_02x03_Odd_Even, SW1 SW_DIP_x01, U1 ATxmega32A4U-AU, U2 TXB0104D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

Commit message: Use better voltage regulator
Parts:
- removed the REF** at (141.6, 76.2)
- added C6: 0.1 uF, Capacitor_SMD:C_0805_2012Metric, F.Cu at (116.2, 89.9)
- added REF**: OSHW-Logo2_9.8x8mm_SilkScreen, Symbol:OSHW-Logo2_9.8x8mm_SilkScreen, F.Cu at (141.6, 76.2)
- C3, C4: value 1uF -> 10uF
- U3: value MIC5504-3.3YM5 -> NCP1117ST33T3G; footprint Package_TO_SOT_SMD:SOT-23-5 -> digikey-footprints:SOT-223
- moved C4 3.85 mm to (129.0, 105.4)
- moved U3 2.29 mm to (126.0, 110.5)
- moved C3 1.80 mm to (122.3, 115.3), turned to 180 degrees
- moved REF** 1.42 mm to (116.2, 111.1)
- moved C5 1.37 mm to (134.6, 111.0), turned to 270 degrees
Connections:
- C3 pad 1: GND -> +5V
- C3 pad 2: +5V -> GND
- U3 pad 1: +5V -> GND
- U3 pad 2: GND -> VCC
Routing:
- net +5V: track 43.5 -> 52.4 mm
- net GND: track 33.1 -> 34.7 mm, vias 15 -> 16
