File: dreaeduino.sch (KiCad schematic (older format))
At the start: 20 parts, among them J1 Conn_01x08_Female, J2 Conn_01x08_Female, J3 Conn_01x08_Female, J4 Conn_01x08_Female, J5 USB_B_Micro, J6 Conn_02x03_Odd_Even, J7 Conn_02x03_Odd_Even, SW1 SW_DIP_x01, U1 ATxmega32A4U-AU, U2 TXB0104D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

Commit message: Use better voltage regulator
Parts:
- removed U3: MIC5504-3.3YM5, Package_TO_SOT_SMD:SOT-23-5, symbol Regulator_Linear:MIC5504-3.3YM5
- added C6: 0.1 uF, Capacitor_SMD:C_0805_2012Metric, symbol Device:C_Small
- added U3: NCP1117ST33T3G, digikey-footprints:SOT-223, symbol dk_PMIC-Voltage-Regulators-Linear:NCP1117ST33T3G
- C1, C2: PartNumber (none) -> 885012007012
- C3, C4: value 1uF -> 10uF; PartNumber (none) -> CC0805ZKY5V6BB106
- C5: Mouser# 581-TAJB106K006TNJ -> (none); PartNumber (none) -> TAJB106K006TNJ
- D1: Mouser# 710-150080GS75000 -> (none); PartNumber (none) -> 150080GS75000
- J5: PartNumber (none) -> 105017-0001
- J6, J7: PartNumber (none) -> 61200621621
- R1: PartNumber (none) -> ERJ-6ENF1002V
- R2: PartNumber (none) -> CRCW0805220RFKEB
- SW1: Mouser# 612-TL3305AF160QG -> (none); PartNumber (none) -> TL3305AF160QG
- U1: PartNumber (none) -> ATxmega32A4-AU
- U2: PartNumber (none) -> TXB0104D
- Y1: Mouser# 732-TX325-26F09Z-AC3 -> (none); PartNumber (none) -> FA-20H 32.0000MF20X-K3
